File: PCB/Next_Make_CPW_2015.brd (EAGLE design)
At the start: 41.6 x 36.8 mm, 6 parts

Commit message: proto board complete
Parts:
- added +LED_10, -LED_10, PB0, PB3: (no value), wirepad:SMD1,27-2,54
Connections:
- new net N$20: +LED_10.1, U$4.PIN_10
- new net N$21: -LED_10.1, U$4.PIN_11
- new net N$22: PB0.1, U$3.PIN_2
- new net N$23: PB3.1, U$3.PIN_4
Routing:
- net N$20: track 0.00 -> 5.08 mm
- net N$21: track 0.00 -> 4.44 mm
- net N$23: track 0.00 -> 3.81 mm
- net N$22: track 0.00 -> 3.81 mm
Other:
- board text added: "10uF"
- board text added: "ATtiny84A"
- board text added: "CPW 2015"
- board text added: "LED Bar"
- board text added: "Next-Make"
- board text added: "Temp Sensor"
Changed lines of the file:
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@@
 <wire x1="41.58" y1="36.82" x2="0" y2="36.82" width="0" layer="20"/>
 <wire x1="0" y1="36.82" x2="0" y2="0" width="0" layer="20"/>
+<text x="17.145" y="23.495" size="1.778" layer="21">ATtiny84A</text>
+<text x="12.065" y="10.795" size="1.778" layer="21">LED Bar</text>
+<text x="40.64" y="33.02" size="2.54" layer="22" rot="MR0">Next-Make</text>
+<text x="40.64" y="29.21" size="2.54" layer="22" rot="MR0">CPW 2015</text>
+<text x="30.48" y="6.35" size="1.27" layer="21">Temp Sensor</text>
+<text x="36.83" y="21.59" size="1.27" layer="21" rot="R90">10uF</text>
 </plain>
 <attributes>
@@
 <element name="U$5" library="Next_Make_CPW_2015" package="TO-92-3" value="MCP9701" x="33.02" y="3.81"/>
 <element name="U$6" library="Next_Make_CPW_2015" package="SMT_MINI_USB" value="USB_MINI" x="6.35" y="36.83" rot="R270"/>
+<element name="+LED_10" library="wirepad" package="SMD1,27-2,54" value="" x="29.21" y="3.81" smashed="yes">
+<attribute name="VALUE" x="29.21" y="3.81" size="0.0254" layer="27"/>
+<attribute name="NAME" x="30.34" y="2.375" size="1.27" layer="25" rot="R180"/>
+</element>
+<element name="-LED_10" library="wirepad" package="SMD1,27-2,54" value="" x="30.48" y="13.335" smashed="yes" rot="R90">
+<attribute name="VALUE" x="30.48" y="13.335" size="0.0254" layer="27" rot="R90"/>
+<attribute name="NAME" x="31.915" y="16.37" size="1.27" layer="25" rot="R270"/>
+</element>
+<element name="PB3" library="wirepad" package="SMD1,27-2,54" value="" x="22.86" y="31.75" smashed="yes">
+<attribute name="VALUE" x="22.86" y="31.75" size="0.0254" layer="27"/>
+<attribute name="NAME" x="24.625" y="34.76" size="1.27" layer="25" rot="R180"/>
+</element>
+<element name="PB0" library="wirepad" package="SMD1,27-2,54" value="" x="27.94" y="31.75" smashed="yes">
+<attribute name="VALUE" x="27.94" y="31.75" size="0.0254" layer="27"/>
+<attribute name="NAME" x="29.705" y="34.76" size="1.27" layer="25" rot="R180"/>
+</element>
 </elements>
 <signals>
@@
 <wire x1="5.08" y1="20.32" x2="5.08" y2="15.24" width="1.016" layer="1"/>
 </signal>
+<signal name="N$20">
+<contactref element="+LED_10" pad="1"/>
+<contactref element="U$4" pad="PIN_10"/>
+<wire x1="27.94" y1="7.62" x2="27.94" y2="3.81" width="1.016" layer="1"/>
+<wire x1="27.94" y1="3.81" x2="29.21" y2="3.81" width="1.016" layer="1"/>
+</signal>
+<signal name="N$21">
+<contactref element="U$4" pad="PIN_11"/>
+<contactref element="-LED_10" pad="1"/>
+<wire x1="27.94" y1="15.24" x2="27.94" y2="13.335" width="1.016" layer="1"/>
+<wire x1="27.94" y1="13.335" x2="30.48" y2="13.335" width="1.016" layer="1"/>
+</signal>
+<signal name="N$22">
+<contactref element="PB0" pad="1"/>
+<contactref element="U$3" pad="PIN_2"/>
+<wire x1="27.94" y1="27.94" x2="27.94" y2="31.75" width="1.016" layer="1"/>
+</signal>
+<signal name="N$23">
+<contactref element="PB3" pad="1"/>
+<contactref element="U$3" pad="PIN_4"/>
+<wire x1="22.86" y1="27.94" x2="22.86" y2="31.75" width="1.016" layer="1"/>
+</signal>
 </signals>
