File: PCB/Next_Make_CPW_2015.sch (EAGLE design)
At the start: 6 parts

Commit message: proto board complete
Parts:
- added +LED_10, -LED_10, PB0, PB3: (no value), wirepad:SMD2
Connections:
- new net N$20: +LED_10.P, U$4.+LED_10
- new net N$21: -LED_10.P, U$4.-LED_10
- new net N$22: PB0.P, U$3.PB0
- new net N$23: PB3.P, U$3.PB3
Changed lines of the file:
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@@
 <part name="GND3" library="supply1" deviceset="GND" device=""/>
 <part name="GND4" library="supply1" deviceset="GND" device=""/>
+<part name="+LED_10" library="wirepad" deviceset="SMD2" device=""/>
+<part name="-LED_10" library="wirepad" deviceset="SMD2" device=""/>
+<part name="PB3" library="wirepad" deviceset="SMD2" device=""/>
+<part name="PB0" library="wirepad" deviceset="SMD2" device=""/>
 </parts>
 <sheets>
@@
 <instance part="GND3" gate="1" x="210.82" y="48.26"/>
 <instance part="GND4" gate="1" x="203.2" y="119.38"/>
+<instance part="+LED_10" gate="1" x="55.88" y="76.2"/>
+<instance part="-LED_10" gate="1" x="106.68" y="71.12" rot="R90"/>
+<instance part="PB3" gate="1" x="144.78" y="99.06"/>
+<instance part="PB0" gate="1" x="144.78" y="109.22"/>
 </instances>
 <busses>
@@
 </segment>
 </net>
+<net name="N$20" class="0">
+<segment>
+<pinref part="+LED_10" gate="1" pin="P"/>
+<pinref part="U$4" gate="G$1" pin="+LED_10"/>
+<wire x1="58.42" y1="76.2" x2="63.5" y2="76.2" width="0.1524" layer="91"/>
+</segment>
+</net>
+<net name="N$21" class="0">
+<segment>
+<pinref part="U$4" gate="G$1" pin="-LED_10"/>
+<pinref part="-LED_10" gate="1" pin="P"/>
+<wire x1="101.6" y1="76.2" x2="106.68" y2="76.2" width="0.1524" layer="91"/>
+<wire x1="106.68" y1="76.2" x2="106.68" y2="73.66" width="0.1524" layer="91"/>
+</segment>
+</net>
+<net name="N$22" class="0">
+<segment>
+<pinref part="PB0" gate="1" pin="P"/>
+<pinref part="U$3" gate="G$1" pin="PB0"/>
+<wire x1="147.32" y1="109.22" x2="152.4" y2="109.22" width="0.1524" layer="91"/>
+</segment>
+</net>
+<net name="N$23" class="0">
+<segment>
+<pinref part="PB3" gate="1" pin="P"/>
+<pinref part="U$3" gate="G$1" pin="PB3"/>
+<wire x1="147.32" y1="99.06" x2="152.4" y2="99.06" width="0.1524" layer="91"/>
+</segment>
+</net>
