File: PCB/Next_Make_CPW_2015_Prototype.sch (EAGLE design)
At the start: 10 parts

Commit message: final board design and updated library
Parts:
- removed +LED_10, -LED_10, PB0, PB3: (no value), wirepad:SMD2
Connections:
- removed net N$22: PB0.P, U$3.PB0
- removed net N$23: PB3.P, U$3.PB3
- removed net N$9: U$1.1K_9, U$4.+LED_9
- net N$20: now also U$1.1K_9, U$4.+LED_9; no longer +LED_10.P
- net N$21: now also U$3.PB0; no longer -LED_10.P
Changed lines of the file:
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@@
 <part name="GND3" library="supply1" deviceset="GND" device=""/>
 <part name="GND4" library="supply1" deviceset="GND" device=""/>
-<part name="+LED_10" library="wirepad" deviceset="SMD2" device=""/>
-<part name="-LED_10" library="wirepad" deviceset="SMD2" device=""/>
-<part name="PB3" library="wirepad" deviceset="SMD2" device=""/>
-<part name="PB0" library="wirepad" deviceset="SMD2" device=""/>
 </parts>
 <sheets>
@@
 <instance part="GND3" gate="1" x="210.82" y="48.26"/>
 <instance part="GND4" gate="1" x="203.2" y="119.38"/>
-<instance part="+LED_10" gate="1" x="55.88" y="76.2"/>
-<instance part="-LED_10" gate="1" x="106.68" y="71.12" rot="R90"/>
-<instance part="PB3" gate="1" x="144.78" y="99.06"/>
-<instance part="PB0" gate="1" x="144.78" y="109.22"/>
 </instances>
 <busses>
@@
 <pinref part="U$4" gate="G$1" pin="+LED_8"/>
 <wire x1="48.26" y1="86.36" x2="63.5" y2="86.36" width="0.1524" layer="91"/>
-</segment>
-</net>
-<net name="N$9" class="0">
-<segment>
-<pinref part="U$1" gate="G$1" pin="1K_9"/>
-<pinref part="U$4" gate="G$1" pin="+LED_9"/>
-<wire x1="48.26" y1="81.28" x2="63.5" y2="81.28" width="0.1524" layer="91"/>
 </segment>
 </net>
@@
 <net name="N$20" class="0">
 <segment>
-<pinref part="+LED_10" gate="1" pin="P"/>
 <pinref part="U$4" gate="G$1" pin="+LED_10"/>
 <wire x1="58.42" y1="76.2" x2="63.5" y2="76.2" width="0.1524" layer="91"/>
+<pinref part="U$1" gate="G$1" pin="1K_9"/>
+<pinref part="U$4" gate="G$1" pin="+LED_9"/>
+<wire x1="48.26" y1="81.28" x2="58.42" y2="81.28" width="0.1524" layer="91"/>
+<wire x1="58.42" y1="81.28" x2="63.5" y2="81.28" width="0.1524" layer="91"/>
+<wire x1="58.42" y1="76.2" x2="58.42" y2="81.28" width="0.1524" layer="91"/>
+<junction x="58.42" y="81.28"/>
 </segment>
 </net>
@@
 <segment>
 <pinref part="U$4" gate="G$1" pin="-LED_10"/>
-<pinref part="-LED_10" gate="1" pin="P"/>
 <wire x1="101.6" y1="76.2" x2="106.68" y2="76.2" width="0.1524" layer="91"/>
 <wire x1="106.68" y1="76.2" x2="106.68" y2="73.66" width="0.1524" layer="91"/>
-</segment>
-</net>
-<net name="N$22" class="0">
-<segment>
-<pinref part="PB0" gate="1" pin="P"/>
+<wire x1="106.68" y1="73.66" x2="137.16" y2="73.66" width="0.1524" layer="91"/>
+<wire x1="137.16" y1="73.66" x2="137.16" y2="109.22" width="0.1524" layer="91"/>
 <pinref part="U$3" gate="G$1" pin="PB0"/>
-<wire x1="147.32" y1="109.22" x2="152.4" y2="109.22" width="0.1524" layer="91"/>
-</segment>
-</net>
-<net name="N$23" class="0">
-<segment>
-<pinref part="PB3" gate="1" pin="P"/>
-<pinref part="U$3" gate="G$1" pin="PB3"/>
-<wire x1="147.32" y1="99.06" x2="152.4" y2="99.06" width="0.1524" layer="91"/>
-</segment>
-</net>
+<wire x1="137.16" y1="109.22" x2="152.4" y2="109.22" width="0.1524" layer="91"/>
+</segment>
+</net>

Commit message: updated board design with instuctions and resistive divider
Parts:
- added R1, R2: 1K, rcl:R-US_M1206
Connections:
- new net N$9: R2.1, U$5.VOUT
- net GND: now also R1.2
- net N$10: now also R1.1, R2.2; no longer U$5.VOUT
Changed lines of the file:
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@@
 <part name="GND3" library="supply1" deviceset="GND" device=""/>
 <part name="GND4" library="supply1" deviceset="GND" device=""/>
+<part name="R1" library="rcl" deviceset="R-US_" device="M1206" value="1K"/>
+<part name="R2" library="rcl" deviceset="R-US_" device="M1206" value="1K"/>
+<part name="GND5" library="supply1" deviceset="GND" device=""/>
 </parts>
 <sheets>
@@
 <instance part="GND3" gate="1" x="210.82" y="48.26"/>
 <instance part="GND4" gate="1" x="203.2" y="119.38"/>
+<instance part="R1" gate="G$1" x="223.52" y="109.22"/>
+<instance part="R2" gate="G$1" x="210.82" y="99.06" rot="R90"/>
+<instance part="GND5" gate="1" x="236.22" y="101.6"/>
 </instances>
 <busses>
@@
 <pinref part="GND4" gate="1" pin="GND"/>
 </segment>
+<segment>
+<pinref part="R1" gate="G$1" pin="2"/>
+<wire x1="228.6" y1="109.22" x2="236.22" y2="109.22" width="0.1524" layer="91"/>
+<wire x1="236.22" y1="109.22" x2="236.22" y2="104.14" width="0.1524" layer="91"/>
+<pinref part="GND5" gate="1" pin="GND"/>
+</segment>
 </net>
 <net name="N$1" class="0">
@@
 <pinref part="U$3" gate="G$1" pin="PA0"/>
 <wire x1="190.5" y1="109.22" x2="210.82" y2="109.22" width="0.1524" layer="91"/>
-<wire x1="210.82" y1="109.22" x2="210.82" y2="63.5" width="0.1524" layer="91"/>
-<pinref part="U$5" gate="G$1" pin="VOUT"/>
-<wire x1="210.82" y1="63.5" x2="218.44" y2="63.5" width="0.1524" layer="91"/>
+<pinref part="R2" gate="G$1" pin="2"/>
+<wire x1="210.82" y1="104.14" x2="210.82" y2="109.22" width="0.1524" layer="91"/>
+<pinref part="R1" gate="G$1" pin="1"/>
+<wire x1="210.82" y1="109.22" x2="218.44" y2="109.22" width="0.1524" layer="91"/>
 </segment>
 </net>
@@
 </segment>
 </net>
+<net name="N$9" class="0">
+<segment>
+<pinref part="U$5" gate="G$1" pin="VOUT"/>
+<wire x1="210.82" y1="63.5" x2="218.44" y2="63.5" width="0.1524" layer="91"/>
+<pinref part="R2" gate="G$1" pin="1"/>
+<wire x1="210.82" y1="63.5" x2="210.82" y2="93.98" width="0.1524" layer="91"/>
+</segment>
+</net>
